Commit message: created setup for dual arm simulation

File: src/robot_urdf/ur5.urdf (robot description, URDF)
Before this commit: robot ur5, 14 links, 13 joints
Joints:
- joint shoulder_lift_joint: origin xyz=0.0 0.0 0.0 rpy=1.570796325 0.0 0.0 -> xyz=0.0 0.0 0.0 rpy=1.570796325 1.570796327 0.0
- joint world_joint: origin xyz=0.0 0.0 0.0 rpy=0.0 0.0 0.0 -> xyz=0.0 0.0 0.0 rpy=0.0 0.0 -1.570796327
- joint wrist_1_joint: origin xyz=-0.39225 0.0 0.10915 rpy=0.0 0.0 0.0 -> xyz=-0.39225 0.0 0.10915 rpy=0.0 0.0 -1.570796327

Commit message: fixed base trajectory generation for newly added UR3e with world to base link transformation.

File: src/robot_urdf/ur5.urdf (robot description, URDF)
Before this commit: robot ur5, 14 links, 13 joints
Joints:
- joint shoulder_lift_joint: origin xyz=0.0 0.0 0.0 rpy=1.570796325 0.0 0.0 -> xyz=0.0 0.0 0.0 rpy=1.570796325 1.570796327 0.0
- joint wrist_1_joint: origin xyz=-0.39225 0.0 0.10915 rpy=0.0 0.0 0.0 -> xyz=-0.39225 0.0 0.10915 rpy=0.0 0.0 -1.570796327
