Commit message: aligned simulation robot configuration to real robots configuration, modified how grasp points are computed (choose the axes mostly aligned to the world's Y axes along which the robots are placed)

File: src/robot_urdf/ur3e.urdf (robot description, URDF)
Before this commit: robot ur3e, 8 links, 7 joints
Joints:
- joint shoulder_lift_joint: origin xyz=0 0 0 rpy=1.570796327 1.570796327 0 -> xyz=0 0 0 rpy=1.570796327 0 0
- joint shoulder_pan_joint: origin xyz=0 0 0.15185 rpy=0 0 -1.570796327 -> xyz=0 0 0.15185 rpy=0 0 0
- joint wrist_1_joint: origin xyz=-0.2132 0 0.13105 rpy=0 0 -1.570796327 -> xyz=-0.2132 0 0.13105 rpy=0 0 0
