Commit message: finished 3d man urdf

File: src/robot_urdf/printed_man.urdf (robot description, URDF)
Before this commit: robot 3Dprinted, 7 links, 6 joints
Links:
- link base_link: geometry visual mesh filename=robot_descriptions/printed_man_description/meshes/visual/li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
- link link_1: geometry visual mesh filename=robot_descriptions/printed_man_description/meshes/visual/li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
- link link_2: geometry visual mesh filename=robot_descriptions/printed_man_description/meshes/visual/li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
- link link_3: geometry visual mesh filename=robot_descriptions/printed_man_description/meshes/visual/li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
- link link_4: geometry visual mesh filename=robot_descriptions/printed_man_description/meshes/visual/li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
- link link_5: geometry visual mesh filename=robot_descriptions/printed_man_description/meshes/visual/li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
- link link_6: geometry visual mesh filename=robot_descriptions/printed_man_description/meshes/visual/li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
Joints:
- joint joint_6: origin xyz=0 -0.07 0 rpy=1.57079632675 0 0 -> xyz=0 -0.0435 0 rpy=1.57079632675 0 0

Commit message: refined 3d printed man urdf and kinematic chain

File: src/robot_urdf/printed_man.urdf (robot description, URDF)
Before this commit: robot 3Dprinted, 7 links, 6 joints
Joints:
- joint joint_6: origin xyz=0 -0.0435 0 rpy=1.57079632675 0 0 -> xyz=0 -0.037 0 rpy=1.57079632675 0 0
